File: PCB/_saved_MCU-STM32F446RET6.sch (KiCad schematic (older format))
At the start: 48 parts, among them J3 20021121-00010C4LF, J4 0475890001-MicroUSBPort, P1 CONN_01X20, P2 CONN_01X20, SW1 B3U-1000P, U3 STM32F446RET6_-_TQFP64, X1 ABM3B8.000MHZB2T, X2 ABS07-32.768KHZ-9-T

Commit message: Board Layout
Board layout started. ESP8285 component placement preliminary complete.
3D parts added and updated for ESP8285. STM32 and SOT32 3/6 pin
packages.
Parts:
- gave numbers to parts that had none: 7
Connections:
- net labels removed: Earth
- wire segments 104 -> 103
- no-connect marks 3 -> 7
