File: PCB/WiFi-ESP8285.sch (KiCad schematic (older format))
At the start: 19 parts, among them SW2 B3U-1000P, T1 1909763-1, U4 ESP8285, X3 FA-128_26.0000MF10Z-AC3

Commit message: Board Layout
Board layout started. ESP8285 component placement preliminary complete.
3D parts added and updated for ESP8285. STM32 and SOT32 3/6 pin
packages.
Connections:
- net GND: now also LED4.2; no longer R21.1
- net at LED4.1: now also R21.1; no longer U4.16 (GOIO4)
- net at R21.2: now also U4.16 (GOIO4); no longer LED4.2
Other:
- moved on the sheet: LED4, R21
Changed lines of the file:
@@
 Wire Wire Line
 	4125 2850 4525 2850
-Wire Wire Line
-	4525 2850 4525 2850
 Connection ~ 4525 2850
 Connection ~ 4125 2850
@@
 	6750 4250 10375 4250
 Wire Wire Line
-	5400 4350 3500 4350
-Wire Wire Line
-	3500 4350 1150 4350
+	1150 4350 3500 4350
+Wire Wire Line
+	3500 4350 5400 4350
 Wire Wire Line
 	3500 4800 3500 4350
@@
 L LTST-C193TBKT-5A LED4
 U 1 1 57EACEB9
-P 4650 3250
-F 0 "LED4" H 4650 2963 60  0000 C CNN
-F 1 "LTST-C193TBKT-5A" H 4650 3069 60  0000 C CNN
-F 2 "PCB_Footprints:LED0603" H 6075 5175 60  0001 C CNN
-F 3 "http://optoelectronics.liteon.com/upload/download/DS22-2004-060/P_100_LTST-C193TBKT-5A.pdf" H 6275 5300 60  0001 C CNN
-F 4 "0.06102 @ 6000" H 4500 3450 60  0001 C CNN "Cost"
-F 5 "8 Sept 2016" H 4600 3550 60  0001 C CNN "Date Created"
-F 6 "8 Sept 2016" H 4700 3650 60  0001 C CNN "Date Modified"
-F 7 "Adam Vadala-Roth" H 4800 3750 60  0001 C CNN "Designer"
-F 8 "0.55mm" H 4900 3850 60  0001 C CNN "Height"
-F 9 "Yes" H 5000 3950 60  0001 C CNN "RhoS?"
-F 10 "Lite-On Inc" H 5100 4050 60  0001 C CNN "MFR"
-F 11 "LTST-C193TBKT-5A" H 5200 4150 60  0001 C CNN "MFR#"
-F 12 "SMT/SMD" H 5300 4250 60  0001 C CNN "Mounting"
-F 13 "2" H 5400 4350 60  0001 C CNN "Pin Count#"
-F 14 "Active" H 5500 4450 60  0001 C CNN "Status"
-F 15 "N/A" H 5600 4550 60  0001 C CNN "Tolerance"
-F 16 "0603 LED" H 5700 4650 60  0001 C CNN "Type"
-F 17 "2.8V Forward Voltage" H 5800 4750 60  0001 C CNN "Voltage"
-F 18 "N/A" H 5900 4850 60  0001 C CNN "Wattage"
-F 19 "N/A" H 6000 4950 60  0001 C CNN "Component-Value"
-F 20 "Blue 470nm LED Indication - Discrete 2.8V 0603 (1608 Metric)" H 6100 5050 60  0001 C CNN "Description"
-	1    4650 3250
+P 3875 3250
+F 0 "LED4" H 3875 2963 60  0000 C CNN
+F 1 "LTST-C193TBKT-5A" H 3875 3069 60  0000 C CNN
+F 2 "PCB_Footprints:LED0603" H 5300 5175 60  0001 C CNN
+F 3 "http://optoelectronics.liteon.com/upload/download/DS22-2004-060/P_100_LTST-C193TBKT-5A.pdf" H 5500 5300 60  0001 C CNN
+F 4 "0.06102 @ 6000" H 3725 3450 60  0001 C CNN "Cost"
+F 5 "8 Sept 2016" H 3825 3550 60  0001 C CNN "Date Created"
+F 6 "8 Sept 2016" H 3925 3650 60  0001 C CNN "Date Modified"
+F 7 "Adam Vadala-Roth" H 4025 3750 60  0001 C CNN "Designer"
+F 8 "0.55mm" H 4125 3850 60  0001 C CNN "Height"
+F 9 "Yes" H 4225 3950 60  0001 C CNN "RhoS?"
+F 10 "Lite-On Inc" H 4325 4050 60  0001 C CNN "MFR"
+F 11 "LTST-C193TBKT-5A" H 4425 4150 60  0001 C CNN "MFR#"
+F 12 "SMT/SMD" H 4525 4250 60  0001 C CNN "Mounting"
+F 13 "2" H 4625 4350 60  0001 C CNN "Pin Count#"
+F 14 "Active" H 4725 4450 60  0001 C CNN "Status"
+F 15 "N/A" H 4825 4550 60  0001 C CNN "Tolerance"
+F 16 "0603 LED" H 4925 4650 60  0001 C CNN "Type"
+F 17 "2.8V Forward Voltage" H 5025 4750 60  0001 C CNN "Voltage"
+F 18 "N/A" H 5125 4850 60  0001 C CNN "Wattage"
+F 19 "N/A" H 5225 4950 60  0001 C CNN "Component-Value"
+F 20 "Blue 470nm LED Indication - Discrete 2.8V 0603 (1608 Metric)" H 5325 5050 60  0001 C CNN "Description"
+	1    3875 3250
 	-1   0    0    1
 $EndComp
@@
 L RC1005F102CS R21
 U 1 1 57EAD2D3
-P 3925 3250
-F 0 "R21" H 3925 3497 60  0000 C CNN
-F 1 "RC1005F102CS" H 3925 3497 60  0001 C CNN
-F 2 "PCB_Footprints:R0402" H 3525 3500 60  0001 C CNN
-F 3 "https://media.digikey.com/pdf/Data%20Sheets/Samsung%20PDFs/RC_Series_ds.pdf" H 3625 3700 60  0001 C CNN
-F 4 "0.00173 @ 5000" H 5475 5200 60  0001 C CNN "Cost"
-F 5 "5 Sept 2016" H 3825 3800 60  0001 C CNN "Date Created"
-F 6 "5 Sept 2016" H 3925 3900 60  0001 C CNN "Date Modified"
-F 7 "Adam Vadala-Roth" H 4025 4000 60  0001 C CNN "Designer"
-F 8 "0.4mm" H 4125 4100 60  0001 C CNN "Height"
-F 9 "Yes" H 4225 4200 60  0001 C CNN "RHoS?"
-F 10 "Samsung Electro-Mechanics America, Inc." H 4325 4300 60  0001 C CNN "MFR"
-F 11 "RC1005F102CS" H 4425 4400 60  0001 C CNN "MFR#"
-F 12 "SMT/SMD" H 4525 4500 60  0001 C CNN "Mounting"
-F 13 "2" H 4625 4600 60  0001 C CNN "Pin Count#"
-F 14 "Active" H 4725 4700 60  0001 C CNN "Status"
-F 15 "%" H 4825 4800 60  0001 C CNN "Tolerance"
-F 16 "passive" H 4925 4900 60  0001 C CNN "Type"
-F 17 "N/A" H 5025 5000 60  0001 C CNN "Voltage"
-F 18 "1/16" H 5125 5100 60  0001 C CNN "Wattage"
-F 19 "1k" H 3925 3391 60  0000 C CNN "Component-Value"
-F 20 "RES SMD 1K OHM 1% 1/16W 0402" H 5325 5300 60  0001 C CNN "Description"
-	1    3925 3250
+P 4600 3250
+F 0 "R21" H 4600 3497 60  0000 C CNN
+F 1 "RC1005F102CS" H 4600 3497 60  0001 C CNN
+F 2 "PCB_Footprints:R0402" H 4200 3500 60  0001 C CNN
+F 3 "https://media.digikey.com/pdf/Data%20Sheets/Samsung%20PDFs/RC_Series_ds.pdf" H 4300 3700 60  0001 C CNN
+F 4 "0.00173 @ 5000" H 6150 5200 60  0001 C CNN "Cost"
+F 5 "5 Sept 2016" H 4500 3800 60  0001 C CNN "Date Created"
+F 6 "5 Sept 2016" H 4600 3900 60  0001 C CNN "Date Modified"
+F 7 "Adam Vadala-Roth" H 4700 4000 60  0001 C CNN "Designer"
+F 8 "0.4mm" H 4800 4100 60  0001 C CNN "Height"
+F 9 "Yes" H 4900 4200 60  0001 C CNN "RHoS?"
+F 10 "Samsung Electro-Mechanics America, Inc." H 5000 4300 60  0001 C CNN "MFR"
+F 11 "RC1005F102CS" H 5100 4400 60  0001 C CNN "MFR#"
+F 12 "SMT/SMD" H 5200 4500 60  0001 C CNN "Mounting"
+F 13 "2" H 5300 4600 60  0001 C CNN "Pin Count#"
+F 14 "Active" H 5400 4700 60  0001 C CNN "Status"
+F 15 "%" H 5500 4800 60  0001 C CNN "Tolerance"
+F 16 "passive" H 5600 4900 60  0001 C CNN "Type"
+F 17 "N/A" H 5700 5000 60  0001 C CNN "Voltage"
+F 18 "1/16" H 5800 5100 60  0001 C CNN "Wattage"
+F 19 "1k" H 4600 3391 60  0000 C CNN "Component-Value"
+F 20 "RES SMD 1K OHM 1% 1/16W 0402" H 6000 5300 60  0001 C CNN "Description"
+	1    4600 3250
 	1    0    0    -1
 $EndComp
@@
 	5400 3250 4900 3250
 Wire Wire Line
-	4225 3250 4400 3250
+	4125 3250 4300 3250
 Wire Wire Line
 	3625 3250 3625 2850

Commit message: Board Size. Routing and Antenna
Board Size tweaked. More signals routed. Next will be pin swapping and
routing finished. Also experimented with importing a PCB antenna design
from bitmap, still can't get it quite right, hopefully nex commit.
Connections:
- net ANTENNA: now reaches T1.1, U4.2 (LNA)
Changed lines of the file:
@@
 ESPTOST_BOOT1
 $Comp
-L GND #PWR35
+L GND #PWR14
 U 1 1 57EA5592
 P 5400 4600
-F 0 "#PWR35" H 5400 4350 50  0001 C CNN
+F 0 "#PWR14" H 5400 4350 50  0001 C CNN
 F 1 "GND" H 5405 4427 50  0000 C CNN
 F 2 "" H 5400 4600 50  0000 C CNN
@@
 $EndComp
 $Comp
-L +3.3V #PWR32
+L +3.3V #PWR11
 U 1 1 57EA55D3
 P 3725 2400
-F 0 "#PWR32" H 3725 2250 50  0001 C CNN
+F 0 "#PWR11" H 3725 2250 50  0001 C CNN
 F 1 "+3.3V" H 3740 2573 50  0000 C CNN
 F 2 "" H 3725 2400 50  0000 C CNN
@@
 $EndComp
 Wire Wire Line
-	2175 2400 2575 2400
-Wire Wire Line
-	2575 2400 2950 2400
-Wire Wire Line
-	2950 2400 3350 2400
-Wire Wire Line
-	3350 2400 3725 2400
-Wire Wire Line
-	3725 2400 4125 2400
-Wire Wire Line
-	4125 2400 4525 2400
-Wire Wire Line
-	4525 2400 5400 2400
+	2175 2400 5400 2400
 Connection ~ 4525 2400
 Connection ~ 4125 2400
@@
 Connection ~ 2575 2400
 Wire Wire Line
-	2175 2850 2575 2850
-Wire Wire Line
-	2575 2850 2950 2850
-Wire Wire Line
-	2950 2850 3350 2850
-Wire Wire Line
-	3350 2850 3625 2850
-Wire Wire Line
-	3625 2850 3725 2850
-Wire Wire Line
-	3725 2850 4125 2850
-Wire Wire Line
-	4125 2850 4525 2850
+	2175 2850 4525 2850
 Connection ~ 4525 2850
 Connection ~ 4125 2850
@@
 Connection ~ 2575 2850
 $Comp
-L GND #PWR31
+L GND #PWR10
 U 1 1 57EA7DCC
 P 3350 2850
-F 0 "#PWR31" H 3350 2600 50  0001 C CNN
+F 0 "#PWR10" H 3350 2600 50  0001 C CNN
 F 1 "GND" H 3355 2677 50  0000 C CNN
 F 2 "" H 3350 2850 50  0000 C CNN
@@
 $EndComp
 Wire Wire Line
-	5400 2400 5400 2500
-Wire Wire Line
-	5400 2500 5400 2600
-Wire Wire Line
-	5400 2600 5400 2700
-Wire Wire Line
-	5400 2700 5400 2800
-Wire Wire Line
-	5400 2800 5400 2900
-Wire Wire Line
-	5400 2900 5400 3000
+	5400 2400 5400 3000
 Connection ~ 5400 2500
 Connection ~ 5400 2600
@@
 	6750 4250 10375 4250
 Wire Wire Line
-	1150 4350 3500 4350
-Wire Wire Line
-	3500 4350 5400 4350
+	1150 4350 5400 4350
 Wire Wire Line
 	3500 4800 3500 4350
@@
 $EndComp
 $Comp
-L GND #PWR30
+L GND #PWR9
 U 1 1 57EABC94
 P 2900 5250
-F 0 "#PWR30" H 2900 5000 50  0001 C CNN
+F 0 "#PWR9" H 2900 5000 50  0001 C CNN
 F 1 "GND" H 2905 5077 50  0000 C CNN
 F 2 "" H 2900 5250 50  0000 C CNN
@@
 $EndComp
 $Comp
-L +3.3V #PWR33
+L +3.3V #PWR12
 U 1 1 57EAC1AB
 P 4100 4800
-F 0 "#PWR33" H 4100 4650 50  0001 C CNN
+F 0 "#PWR12" H 4100 4650 50  0001 C CNN
 F 1 "+3.3V" H 4115 4973 50  0000 C CNN
 F 2 "" H 4100 4800 50  0000 C CNN
@@
 	6750 2400 9250 2400
 $Comp
-L GND #PWR37
+L GND #PWR16
 U 1 1 57EADEB2
 P 9525 2675
-F 0 "#PWR37" H 9525 2425 50  0001 C CNN
+F 0 "#PWR16" H 9525 2425 50  0001 C CNN
 F 1 "GND" H 9530 2502 50  0000 C CNN
 F 2 "" H 9525 2675 50  0000 C CNN
@@
 $EndComp
 $Comp
-L GND #PWR29
+L GND #PWR8
 U 1 1 57EAFC2A
 P 2000 5325
-F 0 "#PWR29" H 2000 5075 50  0001 C CNN
+F 0 "#PWR8" H 2000 5075 50  0001 C CNN
 F 1 "GND" H 2005 5152 50  0000 C CNN
 F 2 "" H 2000 5325 50  0000 C CNN
@@
 $EndComp
 Wire Wire Line
-	1625 5325 1875 5325
-Wire Wire Line
-	1875 5325 2000 5325
-Wire Wire Line
-	2000 5325 2125 5325
-Wire Wire Line
-	2125 5325 2375 5325
+	1625 5325 2375 5325
 Wire Wire Line
 	2125 5225 2125 5325
@@
 $EndComp
 $Comp
-L GND #PWR36
+L GND #PWR15
 U 1 1 57EB2E2B
 P 7350 4600
-F 0 "#PWR36" H 7350 4350 50  0001 C CNN
+F 0 "#PWR15" H 7350 4350 50  0001 C CNN
 F 1 "GND" H 7355 4427 50  0000 C CNN
 F 2 "" H 7350 4600 50  0000 C CNN
@@
 ESP8285 WiFi Radio
 $Comp
-L +3.3V #PWR34
+L +3.3V #PWR13
 U 1 1 57EB7ECC
 P 4300 4175
-F 0 "#PWR34" H 4300 4025 50  0001 C CNN
+F 0 "#PWR13" H 4300 4025 50  0001 C CNN
 F 1 "+3.3V" H 4315 4348 50  0000 C CNN
 F 2 "" H 4300 4175 50  0000 C CNN
@@
 U 1 1 57EBA19F
 P 7050 4600
-F 0 "R23" H 6875 4675 60  0000 C CNN
+F 0 "R23" H 7050 4425 60  0000 C CNN
 F 1 "RC1005F123CS" H 7050 4363 60  0001 C CNN
 F 2 "PCB_Footprints:R0402" H 6650 4850 60  0001 C CNN
@@
 F 17 "N/A" H 8150 6350 60  0001 C CNN "Voltage"
 F 18 "1/16" H 8250 6450 60  0001 C CNN "Wattage"
-F 19 "12K" H 7250 4675 60  0000 C CNN "Component-Value"
+F 19 "12K" H 7050 4500 60  0000 C CNN "Component-Value"
 F 20 "RES SMD 12K OHM 1% 1/16W 0402" H 8450 6650 60  0001 C CNN "Description"
 	1    7050 4600
@@
 U 1 1 57EBBCDB
 P 6100 3550
-F 0 "U4" H 6075 4987 60  0000 C CNN
-F 1 "ESP8285" H 6075 4881 60  0000 C CNN
+F 0 "U4" H 5650 4850 60  0000 C CNN
+F 1 "ESP8285" H 6350 4850 60  0000 C CNN
 F 2 "PCB_Footprints:ESP8285" H 4375 4700 60  0001 C CNN
 F 3 "" H 6100 3550 60  0001 C CNN
@@
 	1    0    0    -1
 $EndComp
+Text Label 7450 2400 0    60   ~ 0
+ANTENNA
 $EndSCHEMATC

Commit message: More routing
more routing completed, but thinking of scraping the current pass
entirely and rechoosing all the pins.
Connections:
- net ESPTOST_BOOT0: now also U4.22 (SD_DATA_0); no longer U4.23 (SD_DATA_1)
- net ESPTOST_BOOT1: now also U4.23 (SD_DATA_1); no longer U4.22 (SD_DATA_0)
Changed lines of the file:
@@
 Text HLabel 1075 3350 0    60   Input ~ 0
 ESP_ST_RST
+Text HLabel 10375 4250 2    60   Input ~ 0
+ESPTOST_BOOT0
 Text HLabel 10375 4350 2    60   Input ~ 0
-ESPTOST_BOOT0
-Text HLabel 10375 4250 2    60   Input ~ 0
 ESPTOST_BOOT1
 $Comp

Commit message: Updates
Changed board size, heavily altered schematic and pinning to be more
efficient. Program mode for ESP8285 is switched to GPIO0 being pulled
high 10k and toggled by STM32. Board at 30mm By 70.5mm. Also switching
to chip antenna next commit, expect updates to libraries.
Parts:
- added R24: RC1005F103CS, PCB_Footprints:R0402, symbol RC1005F103CS
Connections:
- net +3V3: now also R24.1
- net ESP_PGM_MODE: now also U4.15 (GPIO0), R24.2
Changed lines of the file:
@@
 Text HLabel 1150 4350 0    60   Input ~ 0
 STM_ESP_RST
-Text HLabel 7875 3200 2    60   Input ~ 0
+Text HLabel 10375 3650 2    60   Input ~ 0
 ESP_PGM_MODE
 Text HLabel 1075 3350 0    60   Input ~ 0
@@
 	6750 2400 9250 2400
 $Comp
-L GND #PWR16
+L GND #PWR17
 U 1 1 57EADEB2
 P 9525 2675
-F 0 "#PWR16" H 9525 2425 50  0001 C CNN
+F 0 "#PWR17" H 9525 2425 50  0001 C CNN
 F 1 "GND" H 9530 2502 50  0000 C CNN
 F 2 "" H 9525 2675 50  0000 C CNN
@@
 Text Label 7450 2400 0    60   ~ 0
 ANTENNA
+Wire Wire Line
+	6750 3650 10375 3650
+$Comp
+L RC1005F103CS R24
+U 1 1 57FF17D1
+P 8675 3350
+F 0 "R24" V 8569 3438 60  0000 L CNN
+F 1 "RC1005F103CS" V 8675 3438 60  0000 L CNN
+F 2 "PCB_Footprints:R0402" H 8275 3600 60  0001 C CNN
+F 3 "https://media.digikey.com/pdf/Data%20Sheets/Samsung%20PDFs/RC_Series_ds.pdf" H 8375 3800 60  0001 C CNN
+F 4 "0.00173 @ 5000" H 10225 5300 60  0001 C CNN "Cost"
+F 5 "5 Sept 2016" H 8575 3900 60  0001 C CNN "Date Created"
+F 6 "5 Sept 2016" H 8675 4000 60  0001 C CNN "Date Modified"
+F 7 "Adam Vadala-Roth" H 8775 4100 60  0001 C CNN "Designer"
+F 8 "0.4mm" H 8875 4200 60  0001 C CNN "Height"
+F 9 "Yes" H 8975 4300 60  0001 C CNN "RHoS?"
+F 10 "Samsung Electro-Mechanics America, Inc." H 9075 4400 60  0001 C CNN "MFR"
+F 11 "RC1005F103CS" H 9175 4500 60  0001 C CNN "MFR#"
+F 12 "SMT/SMD" H 9275 4600 60  0001 C CNN "Mounting"
+F 13 "2" H 9375 4700 60  0001 C CNN "Pin Count#"
+F 14 "Active" H 9475 4800 60  0001 C CNN "Status"
+F 15 "1%" H 9575 4900 60  0001 C CNN "Tolerance"
+F 16 "passive" H 9675 5000 60  0001 C CNN "Type"
+F 17 "N/A" H 9775 5100 60  0001 C CNN "Voltage"
+F 18 "1/16" H 9875 5200 60  0001 C CNN "Wattage"
+F 19 "10k" V 8781 3438 60  0000 L CNN "Component-Value"
+F 20 "RES SMD 10K OHM 1% 1/16W 0402" H 10075 5400 60  0001 C CNN "Description"
+	1    8675 3350
+	0    1    1    0
+$EndComp
+Connection ~ 8675 3650
+$Comp
+L +3.3V #PWR16
+U 1 1 57FF1E19
+P 8675 3050
+F 0 "#PWR16" H 8675 2900 50  0001 C CNN
+F 1 "+3.3V" H 8690 3223 50  0000 C CNN
+F 2 "" H 8675 3050 50  0000 C CNN
+F 3 "" H 8675 3050 50  0000 C CNN
+	1    8675 3050
+	1    0    0    -1
+$EndComp
 $EndSCHEMATC

Commit message: Board Finished
Board finished
Parts:
- added ANT1: Inverted_F_PCB_Antenna, PCB_Footprints:PCB_IF_ANT_2.4G, symbol Inverted_F_PCB_Antenna
- added C29: 600L5R6BT200T, PCB_Footprints:C0402, symbol 600L5R6BT200T
- added R25, R26: ERJ-2GE0R00X, PCB_Footprints:R0402, symbol ERJ-2GE0R00X
Connections:
- net ANTENNA: now also C29.2, R25.1, R26.1; no longer T1.1, U4.2 (LNA)
- net GND: now also ANT1.2
- new net ANT_F: ANT1.1, R25.2
- new net ANT_UM: R26.2, T1.1
- new net LNA: C29.1, U4.2 (LNA)
Other:
- moved on the sheet: T1
