File: PCB/MCU-STM32F446RET6.sch (KiCad schematic (older format))
At the start: 48 parts, among them J3 20021121-00010C4LF, J4 0475890001-MicroUSBPort, P1 CONN_01X18, P2 CONN_01X18, SW1 B3U-1000P, U3 STM32F446RET6_-_TQFP64, X1 ABM3B8.000MHZB2T, X2 ABS07-32.768KHZ-9-T

Commit message: Board Finished
Board finished
Changed lines of the file:
@@
 $EndComp
 $Comp
-L GND #PWR24
+L GND #PWR25
 U 1 1 57D43B63
 P 2025 6725
-F 0 "#PWR24" H 2025 6475 50  0001 C CNN
+F 0 "#PWR25" H 2025 6475 50  0001 C CNN
 F 1 "GND" H 2025 6575 50  0000 C CNN
 F 2 "" H 2025 6725 50  0000 C CNN
@@
 $EndComp
 $Comp
-L GND #PWR26
+L GND #PWR27
 U 1 1 57D43E04
 P 2350 7425
-F 0 "#PWR26" H 2350 7175 50  0001 C CNN
+F 0 "#PWR27" H 2350 7175 50  0001 C CNN
 F 1 "GND" H 2350 7275 50  0000 C CNN
 F 2 "" H 2350 7425 50  0000 C CNN
@@
 $EndComp
 $Comp
-L +3.3V #PWR20
+L +3.3V #PWR21
 U 1 1 57D443BB
 P 1475 6275
-F 0 "#PWR20" H 1475 6125 50  0001 C CNN
+F 0 "#PWR21" H 1475 6125 50  0001 C CNN
 F 1 "+3.3V" H 1475 6415 50  0000 C CNN
 F 2 "" H 1475 6275 50  0000 C CNN
@@
 $EndComp
 $Comp
-L +3.3V #PWR21
+L +3.3V #PWR22
 U 1 1 57D444DD
 P 1475 6975
-F 0 "#PWR21" H 1475 6825 50  0001 C CNN
+F 0 "#PWR22" H 1475 6825 50  0001 C CNN
 F 1 "+3.3V" H 1475 7115 50  0000 C CNN
 F 2 "" H 1475 6975 50  0000 C CNN
@@
 $EndComp
 $Comp
-L GND #PWR35
+L GND #PWR36
 U 1 1 57D449FF
 P 5950 5575
-F 0 "#PWR35" H 5950 5325 50  0001 C CNN
+F 0 "#PWR36" H 5950 5325 50  0001 C CNN
 F 1 "GND" H 5950 5425 50  0000 C CNN
 F 2 "" H 5950 5575 50  0000 C CNN
@@
 $EndComp
 $Comp
-L +3.3V #PWR33
+L +3.3V #PWR34
 U 1 1 57D45F91
 P 5350 4975
-F 0 "#PWR33" H 5350 4825 50  0001 C CNN
+F 0 "#PWR34" H 5350 4825 50  0001 C CNN
 F 1 "+3.3V" H 5350 5115 50  0000 C CNN
 F 2 "" H 5350 4975 50  0000 C CNN
@@
 $EndComp
 $Comp
-L GND #PWR31
+L GND #PWR32
 U 1 1 57D46AC6
 P 4725 7425
-F 0 "#PWR31" H 4725 7175 50  0001 C CNN
+F 0 "#PWR32" H 4725 7175 50  0001 C CNN
 F 1 "GND" H 4725 7275 50  0000 C CNN
 F 2 "" H 4725 7425 50  0000 C CNN
@@
 $EndComp
 $Comp
-L GND #PWR32
+L GND #PWR33
 U 1 1 57D47BC2
 P 5125 7425
-F 0 "#PWR32" H 5125 7175 50  0001 C CNN
+F 0 "#PWR33" H 5125 7175 50  0001 C CNN
 F 1 "GND" H 5125 7275 50  0000 C CNN
 F 2 "" H 5125 7425 50  0000 C CNN
@@
 $EndComp
 $Comp
-L GND #PWR23
+L GND #PWR24
 U 1 1 57D49635
 P 1975 5800
-F 0 "#PWR23" H 1975 5550 50  0001 C CNN
+F 0 "#PWR24" H 1975 5550 50  0001 C CNN
 F 1 "GND" H 1975 5650 50  0000 C CNN
 F 2 "" H 1975 5800 50  0000 C CNN
@@
 $EndComp
 $Comp
-L GND #PWR36
+L GND #PWR37
 U 1 1 57D4B2EA
 P 6850 4450
-F 0 "#PWR36" H 6850 4200 50  0001 C CNN
+F 0 "#PWR37" H 6850 4200 50  0001 C CNN
 F 1 "GND" H 6850 4300 50  0000 C CNN
 F 2 "" H 6850 4450 50  0000 C CNN
@@
 $EndComp
 $Comp
-L GND #PWR30
+L GND #PWR31
 U 1 1 57D4C07E
 P 2625 6400
-F 0 "#PWR30" H 2625 6150 50  0001 C CNN
+F 0 "#PWR31" H 2625 6150 50  0001 C CNN
 F 1 "GND" H 2625 6250 50  0000 C CNN
 F 2 "" H 2625 6400 50  0000 C CNN
@@
 $EndComp
 $Comp
-L GND #PWR37
+L GND #PWR38
 U 1 1 57D53F54
 P 8325 1150
-F 0 "#PWR37" H 8325 900 50  0001 C CNN
+F 0 "#PWR38" H 8325 900 50  0001 C CNN
 F 1 "GND" H 8325 1000 50  0000 C CNN
 F 2 "" H 8325 1150 50  0000 C CNN
@@
 $EndComp
 $Comp
-L GND #PWR45
+L GND #PWR46
 U 1 1 57D5C6D5
 P 10225 4150
-F 0 "#PWR45" H 10225 3900 50  0001 C CNN
+F 0 "#PWR46" H 10225 3900 50  0001 C CNN
 F 1 "GND" H 10225 4000 50  0000 C CNN
 F 2 "" H 10225 4150 50  0000 C CNN
@@
 $EndComp
 $Comp
-L GND #PWR43
+L GND #PWR44
 U 1 1 57D5C856
 P 9525 4250
-F 0 "#PWR43" H 9525 4000 50  0001 C CNN
+F 0 "#PWR44" H 9525 4000 50  0001 C CNN
 F 1 "GND" H 9525 4100 50  0000 C CNN
 F 2 "" H 9525 4250 50  0000 C CNN
@@
 $EndComp
 $Comp
-L GND #PWR44
+L GND #PWR45
 U 1 1 57D5C8C7
 P 9725 3150
-F 0 "#PWR44" H 9725 2900 50  0001 C CNN
+F 0 "#PWR45" H 9725 2900 50  0001 C CNN
 F 1 "GND" H 9725 3000 50  0000 C CNN
 F 2 "" H 9725 3150 50  0000 C CNN
@@
 $EndComp
 $Comp
-L GND #PWR41
+L GND #PWR42
 U 1 1 57D5FF55
 P 9125 3500
-F 0 "#PWR41" H 9125 3250 50  0001 C CNN
+F 0 "#PWR42" H 9125 3250 50  0001 C CNN
 F 1 "GND" H 9125 3350 50  0000 C CNN
 F 2 "" H 9125 3500 50  0000 C CNN
@@
 $EndComp
 $Comp
-L +3.3V #PWR39
+L +3.3V #PWR40
 U 1 1 57D61D70
 P 8400 5125
-F 0 "#PWR39" H 8400 4975 50  0001 C CNN
+F 0 "#PWR40" H 8400 4975 50  0001 C CNN
 F 1 "+3.3V" H 8400 5265 50  0000 C CNN
 F 2 "" H 8400 5125 50  0000 C CNN
@@
 STM32F446RET6 Main MCU
 $Comp
-L +3.3V #PWR29
+L +3.3V #PWR30
 U 1 1 57D91770
 P 2625 5950
-F 0 "#PWR29" H 2625 5800 50  0001 C CNN
+F 0 "#PWR30" H 2625 5800 50  0001 C CNN
 F 1 "+3.3V" H 2625 6090 50  0000 C CNN
 F 2 "" H 2625 5950 50  0000 C CNN
@@
 $EndComp
 $Comp
-L GND #PWR38
+L GND #PWR39
 U 1 1 57DDB978
 P 8325 6225
-F 0 "#PWR38" H 8325 5975 50  0001 C CNN
+F 0 "#PWR39" H 8325 5975 50  0001 C CNN
 F 1 "GND" H 8325 6075 50  0000 C CNN
 F 2 "" H 8325 6225 50  0000 C CNN
@@
 HEARTBEAT
 $Comp
-L GND #PWR42
+L GND #PWR43
 U 1 1 57E11BCD
 P 9375 1275
-F 0 "#PWR42" H 9375 1025 50  0001 C CNN
+F 0 "#PWR43" H 9375 1025 50  0001 C CNN
 F 1 "GND" H 9375 1125 50  0000 C CNN
 F 2 "" H 9375 1275 50  0000 C CNN
@@
 $EndComp
 $Comp
-L +3.3V #PWR40
+L +3.3V #PWR41
 U 1 1 57E391E0
 P 8900 775
-F 0 "#PWR40" H 8900 625 50  0001 C CNN
+F 0 "#PWR41" H 8900 625 50  0001 C CNN
 F 1 "+3.3V" H 8900 915 50  0000 C CNN
 F 2 "" H 8900 775 50  0000 C CNN
@@
 NoConn ~ 3175 4300
 $Comp
-L GND #PWR28
+L GND #PWR29
 U 1 1 57EDFE20
 P 2550 725
-F 0 "#PWR28" H 2550 475 50  0001 C CNN
+F 0 "#PWR29" H 2550 475 50  0001 C CNN
 F 1 "GND" H 2550 575 50  0000 C CNN
 F 2 "" H 2550 725 50  0000 C CNN
@@
 Text Label 6600 3550 0    60   ~ 0
 PC12
-Text Label 1175 1475 0    60   ~ 0
+Text Label 1175 1575 0    60   ~ 0
 PC10
-Text Label 1175 1675 0    60   ~ 0
+Text Label 1175 1775 0    60   ~ 0
 PC12
 $Comp
-L GND #PWR34
+L GND #PWR35
 U 1 1 57EF642A
 P 5350 6025
-F 0 "#PWR34" H 5350 5775 50  0001 C CNN
+F 0 "#PWR35" H 5350 5775 50  0001 C CNN
 F 1 "GND" H 5350 5875 50  0000 C CNN
 F 2 "" H 5350 6025 50  0000 C CNN
@@
 Text Label 6550 1950 0    60   ~ 0
 PB5
+Text Label 1175 2275 0    60   ~ 0
+PB9
 Text Label 1175 2175 0    60   ~ 0
-PB9
+PB8
 Text Label 1175 2075 0    60   ~ 0
-PB8
+PB7
 Text Label 1175 1975 0    60   ~ 0
-PB7
+PB6
 Text Label 1175 1875 0    60   ~ 0
-PB6
-Text Label 1175 1775 0    60   ~ 0
 PB5
 $Comp
-L +3.3V #PWR27
+L +3.3V #PWR28
 U 1 1 57EFBBDD
 P 2400 775
-F 0 "#PWR27" H 2400 625 50  0001 C CNN
+F 0 "#PWR28" H 2400 625 50  0001 C CNN
 F 1 "+3.3V" H 2400 915 50  0000 C CNN
 F 2 "" H 2400 775 50  0000 C CNN
@@
 Text Label 6550 3150 0    60   ~ 0
 PC8
-Text Label 1175 2575 0    60   ~ 0
+Text Label 2225 1275 0    60   ~ 0
 PC9
 Text Label 2225 1375 0    60   ~ 0
@@
 Text Label 4250 2650 0    60   ~ 0
 PA12
-Text Label 2225 1275 0    60   ~ 0
+Text Label 2225 1175 0    60   ~ 0
 PA8
-Text Label 2225 1175 0    60   ~ 0
+Text Label 1175 1175 0    60   ~ 0
 PA9
-Text Label 1175 1175 0    60   ~ 0
+Text Label 1175 1275 0    60   ~ 0
 PA10
-Text Label 1175 1275 0    60   ~ 0
+Text Label 1175 1375 0    60   ~ 0
 PA11
-Text Label 1175 1375 0    60   ~ 0
+Text Label 1175 1475 0    60   ~ 0
 PA12
 Wire Wire Line
@@
 Wire Wire Line
 	1150 3450 4625 3450
-Text Label 1175 1575 0    60   ~ 0
+Text Label 1175 1675 0    60   ~ 0
 PC11
 Text Label 4400 3250 0    60   ~ 0
@@
 Text Label 4400 3150 0    60   ~ 0
 PC0
+Text Label 1175 2575 0    60   ~ 0
+PC1
 Text Label 1175 2475 0    60   ~ 0
-PC1
-Text Label 1175 2375 0    60   ~ 0
 PC0
 Wire Wire Line
@@
 Text Label 6600 3650 0    60   ~ 0
 PC13
-Text Label 1175 2275 0    60   ~ 0
+Text Label 1175 2375 0    60   ~ 0
 PC13
 Text Label 6525 1450 0    60   ~ 0
@@
 	2275 2675 2275 2875
 $Comp
-L GND #PWR25
+L GND #PWR26
 U 1 1 57EEC925
 P 2275 2875
-F 0 "#PWR25" H 2275 2625 50  0001 C CNN
+F 0 "#PWR26" H 2275 2625 50  0001 C CNN
 F 1 "GND" H 2275 2725 50  0000 C CNN
 F 2 "" H 2275 2875 50  0000 C CNN
@@
 	1200 2675 1200 3100
 $Comp
-L GND #PWR18
+L GND #PWR19
 U 1 1 57EED0C8
 P 1200 3100
-F 0 "#PWR18" H 1200 2850 50  0001 C CNN
+F 0 "#PWR19" H 1200 2850 50  0001 C CNN
 F 1 "GND" H 1200 2950 50  0000 C CNN
 F 2 "" H 1200 3100 50  0000 C CNN
@@
 PA5
 $Comp
-L GND #PWR22
+L GND #PWR23
 U 1 1 57EF36B3
 P 1500 725
-F 0 "#PWR22" H 1500 475 50  0001 C CNN
+F 0 "#PWR23" H 1500 475 50  0001 C CNN
 F 1 "GND" H 1500 575 50  0000 C CNN
 F 2 "" H 1500 725 50  0000 C CNN
@@
 $EndComp
 $Comp
-L +3.3V #PWR19
+L +3.3V #PWR20
 U 1 1 57EF36B9
 P 1350 775
-F 0 "#PWR19" H 1350 625 50  0001 C CNN
+F 0 "#PWR20" H 1350 625 50  0001 C CNN
 F 1 "+3.3V" H 1350 915 50  0000 C CNN
 F 2 "" H 1350 775 50  0000 C CNN
@@
 	1350 1075 1400 1075
 Wire Wire Line
+	1125 2475 1400 2475
+Wire Wire Line
+	1125 2575 1400 2575
+Wire Wire Line
+	1125 2275 1400 2275
+Wire Wire Line
 	1125 2375 1400 2375
 Wire Wire Line
-	1125 2475 1400 2475
+	1125 2075 1400 2075
 Wire Wire Line
 	1125 2175 1400 2175
 Wire Wire Line
-	1125 2275 1400 2275
+	1125 1875 1400 1875
 Wire Wire Line
 	1125 1975 1400 1975
 Wire Wire Line
-	1125 2075 1400 2075
-Wire Wire Line
 	1125 1775 1400 1775
 Wire Wire Line
-	1125 1875 1400 1875
+	1125 1575 1400 1575
 Wire Wire Line
 	1125 1675 1400 1675
 Wire Wire Line
+	1125 1375 1400 1375
+Wire Wire Line
 	1125 1475 1400 1475
 Wire Wire Line
-	1125 1575 1400 1575
-Wire Wire Line
 	1125 1275 1400 1275
-Wire Wire Line
-	1125 1375 1400 1375
-Wire Wire Line
-	1125 1175 1400 1175
-Wire Wire Line
-	1125 2575 1400 2575
 $Comp
 L CONN_01X18 P1
@@
 Wire Wire Line
 	2450 1675 2125 1675
+Wire Wire Line
+	1125 1175 1400 1175
 $EndSCHEMATC
